File: 3x3 Minibadge Display/Minibadge Holder 3x3.kicad_sch (KiCad schematic)
At the start: 32 parts, among them J1 TYPE-C-31-M-17, SW1 SW_SPDT, U1 AP2112K-3.3, U2 74HC4060, U3 TPM8837C

Commit message: r3 (on/off, graphics, laser cut files)
Parts:
- added SW1: ON/OFF, Button_Switch_SMD:SW_SPDT_PCM12, symbol Switch:SW_SPDT
- D1, D2, D3: footprint LED_SMD:LED_1206_3216Metric_Pad1.42x1.75mm_HandSolder -> LED_SMD:LED_1206_3216Metric_ReverseMount_Hole1.8x2.4mm
- R3, R7: value 5.1k -> 5.1kΩ
- R5: value 20k -> 20kΩ
- SW2: renamed from SW1; value SW_SPDT -> CLOCK SPEED
- U2: value 74HC4060 -> 74HC4060D; footprint Package_SO:SSOP-16_5.3x6.2mm_P0.65mm -> 74LV4060D,118:74LV4060D118
- renumbered J1 to USB1
Connections:
- net VBUS: now also SW1.2 (B); no longer U1.3 (EN)
- new net: SW1.1 (A), U1.3 (EN)
Other:
- note added: "3.3v Regulator + on/off"
- note removed: "3.3v Regulator"
- moved on the sheet: C1, C2, C3, C4, D1, D2, D3, MB1, MB2, MB3, MB4, MB5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
