File: Julia Reagan/Julia Reagan.kicad_pcb (KiCad board)
At the start: 2 copper layers, 40.6 x 37.7 mm, 7 parts

Commit message: Update Julia minibadge
Parts:
- removed mouse-bite-2.54mm-slot (x2): VAL**, Panelization.pretty-master:mouse-bite-2.54mm-slot
- D1, D2: footprint LED_SMD:LED_0805_2012Metric -> LED_SMD:LED_1206_3216Metric; moved to B.Cu
- R1, R2: footprint Resistor_SMD:R_0603_1608Metric -> Resistor_SMD:R_1206_3216Metric; moved to B.Cu
- moved D2 29.0 mm to (89.9, 92.6)
- moved R2 25.1 mm to (84.3, 92.5), turned to 0 degrees
- moved D1 19.7 mm to (101.5, 83.1)
- moved R1 15.6 mm to (95.9, 83.1), turned to 0 degrees
Routing:
- net +3.3V: track 58.4 -> 17.3 mm
- net GND: track 15.7 -> 15.0 mm
- net Net-(D2-A): track 2.19 -> 2.80 mm
- net Net-(D1-A): track 2.19 -> 2.76 mm
- removed copper zone on B.Cu, net GND
Other:
- board size 40.6 x 37.7 mm -> 40.6 x 25.4 mm
- board text removed: "+3.3v"
- board text removed: "2025"
- board text removed: "GND"
- board text removed: "Pips"
- board text removed: "XoYdiuM"
