File: Microbadge Minibadge/Microbadge Minibadge.kicad_pcb (KiCad board)
At the start: 2 copper layers, 20 x 20 mm, 7 parts

Commit message: R2 Microbadge Minibadge
Parts:
- removed the MCB6 at (116.5, 114.0)
- added MCB1: Microbadge V2 Full, Microbadge V2:Microbadge_V2_full_round_socket_reflective_nosilk_GND, F.Cu at (103.9, 107.0)
- MCB2, MCB3, MCB4, MCB5: footprint Microbadge V2:Microbadge_V2_full_round_socket_reflective_GND -> Microbadge V2:Microbadge_V2_full_round_socket_reflective_nosilk_GND
- MCB6: renamed from MCB1; footprint Microbadge V2:Microbadge_V2_full_round_socket_reflective_GND -> Microbadge V2:Microbadge_V2_full_round_socket_reflective_nosilk_GND
- moved MCB6 14.4 mm to (117.1, 113.8)
- moved MCB4 0.59 mm to (103.9, 113.8)
- moved MCB3 0.58 mm to (117.1, 107.0)
- moved MCB5 0.18 mm to (110.5, 113.8)
Routing:
- net GND: track 98.8 -> 0.00 mm
- net +3.3V: track 72.5 -> 0.00 mm
- net SDA: track 50.9 -> 0.00 mm, vias 8 -> 0
- net SCL: track 45.5 -> 0.00 mm, vias 6 -> 0
- net CLK: track 42.8 -> 0.00 mm, vias 2 -> 0
- net +VBATT: track 37.5 -> 0.00 mm, vias 1 -> 0
- added copper zone on In2.Cu, net +3.3V
- added copper zone on In1.Cu, net +VBATT
- added copper zone on B.Cu, net CLK
- added copper zone on F.Cu, net GND
Other:
- copper layers 2 -> 4
- board text added: "MICROBADGE"
- board text added: "SAINTCON"
- board text added: "SAINTCON MICROBADGE MINIBADGE (V2)"
- board text added: "SUPPORTS 6X V2 MICROBADGES"
- board text removed: "SAINTCON Microbadge"
