File: Microbadge Minibadge/Microbadge Minibadge.kicad_sch (KiCad schematic)
At the start: 7 parts

Commit message: R2 Microbadge Minibadge
Parts:
- MCB1, MCB2, MCB3, MCB4, MCB5, MCB6: footprint Microbadge V2:Microbadge_V2_full_round_socket_reflective_GND -> Microbadge V2:Microbadge_V2_full_round_socket_reflective_nosilk_GND
Changed lines of the file:
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@@
 			)
 		)
-		(property "Footprint" "Microbadge V2:Microbadge_V2_full_round_socket_reflective_GND"
+		(property "Footprint" "Microbadge V2:Microbadge_V2_full_round_socket_reflective_nosilk_GND"
 			(at 54.61 63.5 0)
 			(effects
@@
 			)
 		)
-		(property "Footprint" "Microbadge V2:Microbadge_V2_full_round_socket_reflective_GND"
+		(property "Footprint" "Microbadge V2:Microbadge_V2_full_round_socket_reflective_nosilk_GND"
 			(at 107.95 88.9 0)
 			(effects
@@
 			)
 		)
-		(property "Footprint" "Microbadge V2:Microbadge_V2_full_round_socket_reflective_GND"
+		(property "Footprint" "Microbadge V2:Microbadge_V2_full_round_socket_reflective_nosilk_GND"
 			(at 54.61 88.9 0)
 			(effects
@@
 			)
 		)
-		(property "Footprint" "Microbadge V2:Microbadge_V2_full_round_socket_reflective_GND"
+		(property "Footprint" "Microbadge V2:Microbadge_V2_full_round_socket_reflective_nosilk_GND"
 			(at 107.95 63.5 0)
 			(effects
@@
 			)
 		)
-		(property "Footprint" "Microbadge V2:Microbadge_V2_full_round_socket_reflective_GND"
+		(property "Footprint" "Microbadge V2:Microbadge_V2_full_round_socket_reflective_nosilk_GND"
 			(at 54.61 114.3 0)
 			(effects
@@
 			)
 		)
-		(property "Footprint" "Microbadge V2:Microbadge_V2_full_round_socket_reflective_GND"
+		(property "Footprint" "Microbadge V2:Microbadge_V2_full_round_socket_reflective_nosilk_GND"
 			(at 107.95 114.3 0)
 			(effects
