File: XIAO ESP minibadge/XIAO ESP minibadge.kicad_pcb (KiCad board)
At the start: 2 copper layers, 20.3 x 22.9 mm, 8 parts, among them U1 XIAO-ESP32-S3-DIP

Commit message: updates
Other:
- board text added: "Pips801 2026"
- board text added: "XIAO ESP32"

Commit message: XIAO update
Routing:
- net /X_3V3: track 12.8 -> 0.00 mm
- net /X_VBUS: track 12.0 -> 0.00 mm
- net Net-(D2-A): track 3.41 -> 0.00 mm
- net Net-(D1-A): track 3.41 -> 0.00 mm
- net VBUS: track 2.93 -> 0.00 mm
- added copper zone on F.Cu, net /X_3V3
- added copper zone on F.Cu, net /X_VBUS
- added copper zone on B.Cu, net Net-(D1-A)
- added copper zone on B.Cu, net Net-(D2-A)
- added copper zone on B.Cu, net VBUS
Other:
- board size 20.3 x 22.9 mm -> 20.3 x 22.1 mm
- board text added: "Pips801"
- board text removed: "Back of board"
- board text removed: "Pips801 2026"
- board text removed: "XIAO ESP32"
