File: Charge your phone Minibadge/Charge your phone Minibadge.kicad_sch (KiCad schematic)
At the start: 17 parts, among them J1 USB-C DFP, U1 MT3608, U2 TPS255x

Commit message: Finalize rev1
Parts:
- removed C4: 0.1μF, Capacitor_SMD:C_0603_1608Metric, symbol Device:C_Small
- D1: LCSC Part # (none) -> C7420328
- L1: footprint Inductor_SMD:L_Wuerth_MAPI-3020 -> Inductor_SMD:L_Taiyo-Yuden_MD-4040; Alt1 LCSC Part # (none) -> C7433093; Alt2 LCSC Part # (none) -> C17701300; LCSC Part # (none) -> C602031
- R1: value ? -> 750kΩ; LCSC Part # (none) -> C23240
- R2: value ? -> 100kΩ; LCSC Part # (none) -> C25803
- R4: value 59kΩ* -> 51kΩ; LCSC Part # (none) -> C23196
- U1: LCSC Part # (none) -> C84817
- U2: value TPS255x -> TPS2552; LCSC Part # (none) -> C46506
Connections:
- net GND: now also U2.3 (EN)
Other:
- note added: "5.1kΩ = ~510mA ILIM"
- note added: "750/100kΩ = 5.1V output"
- note removed: "Confirm EN pin behavior"
- note removed: "Confirm Feedback resistors for 5.1V"
- note removed: "Confirm ILIM Value for ~500mA"
- company: (none) -> Pips Engineering
- title: (none) -> USB-C charger minibadge
- moved on the sheet: C2, C3, C5, D1, J1, L1, R1, R2, R5, R6, U1
